Commit message: robothome

File: autodex/planner/src/curobo/content/assets/robot/inspire_description/inspire_left_floating.urdf (robot description, URDF)
Before this commit: robot inspire_floating, 26 links, 25 joints
Joints:
- joint left_middle_2_joint: mimic joint=left_middle_1_joint multiplier=1.05 offset=0 -> joint=left_middle_1_joint multiplier=0.88 offset=0.15

File: src/validation/robothome/fr3_inspire_left.urdf (robot description, URDF)
Before this commit: robot fr3_inspire_left, 24 links, 23 joints
Joints:
- joint left_middle_2_joint: mimic joint=left_middle_1_joint multiplier=1.05 offset=0 -> joint=left_middle_1_joint multiplier=0.88 offset=0.15
